File: max2769test.kicad_sch (KiCad schematic)
At the start: 76 parts, among them J1 Conn_Coaxial, J3 Conn_01x03_Socket, J4 Conn_01x05_Pin, SW1 SW_Push, U1 MAX2769B, U2 ICE40UP5K-SG48ITR, U3 STM32C051K6T6, U4 TPS7A20, U5 TPS7A20, U6 TX22-M010S, U7 TPS7A20, U8 RTL8211FD

Commit message: work on ethernet phy layout
Parts:
- added C41, C43, C45, C47, C49: 4.7u, symbol Device:C_Small
- added C42, C44, C46, C48, C50: 100n, symbol Device:C_Small
- added D1, D2, D3: LED, symbol Device:LED
- added R10, R8: 4.7k, RF_Module:Digi_XBee_SMT, symbol Device:R_Small
- added R11, R9: 510, RF_Module:Digi_XBee_SMT, symbol Device:R_Small
- added R12: 4.7k, symbol Device:R_Small
- added R13: 510, symbol Device:R_Small
- added R7: 1.5k, symbol Device:R_Small
- added TP19, TP20, TP21: TestPoint, symbol Connector:TestPoint
- R4, R5: footprint Resistor_THT:R_Array_SIP4 -> (none)
Connections:
- net PHY_LDO_OUT_A is gone; now on net PHY_LDO_OUT: U8.3 (AVDD10), U8.38 (AVDD10), U8.8 (AVDD10)
- net PHY_LDO_OUT_D is gone; now on net PHY_LDO_OUT: U8.21 (DVDD10)
- net GND: now also C41.2, C42.2, C43.2, C44.2, C45.2, C46.2, C47.2, C48.2, C49.2, C50.2, R10.2, R11.2, R8.2, R9.2
- net ICE40_P2V85: now also U2.33 (VCCIO_0)
- net P1V2: now also TP19.1
- net PHY_LDO_OUT: now also C41.1, C42.1, C43.1, C44.1, C45.1, C46.1, C47.1, C48.1, C49.1, C50.1, TP20.1
- net PHY_VDDIO: now also R6.2, R7.1; no longer R6.1
- net PHY_RXC: now reaches R4.1
- net PHY_RXC: now also U2.37 (IOT_45a_G1), U8.27 (RXC/PHYAD1); no longer U8.26 (RXCTL/PHYAD2)
- net PHY_MDIO: now reaches U3.14 (PA7)
- net PHY_MDIO: now also U8.14 (MDIO), R7.2
- net PHY_MDC: now reaches U3.18 (PA8)
- net PHY_MDC: now also U8.13 (MDC)
- net PHY_NRST: now reaches U3.27 (PB3)
- net PHY_NRST: now also U8.12 (PHYRSTB)
- net PHY_RXD3: now reaches U8.22 (RXD3/PHYAD0)
- net PHY_RXD3: now also R6.1, U2.34 (IOT_44b); no longer R6.2
- net PHY_TXD3: now reaches U8.15 (TXD3)
- net PHY_TXD3: now also U2.38 (IOT_50b)
- net PHY_TXD: now reaches U8.16 (TXD2)
- net PHY_TXD1: now reaches U8.17 (TXD1)
- net PHY_TXD1: now also U2.42 (IOT_51a)
- net PHY_TXD0: now reaches U8.18 (TXD0)
- net PHY_TXD0: now also U2.43 (IOT_49a)
- net PHY_TXCTL: now reaches U8.19 (TXCTL)
- net PHY_TXCTL: now also U2.36 (IOT_48b)
- net PHY_TXC: now reaches U8.20 (TXC)
- net PHY_TXC: now also U2.35 (IOT_46b_G0)
- net PHY_RXD2: now reaches U8.23 (RXD2/PLLOFF)
- net PHY_RXD2: now also U2.32 (IOT_43a)
- net PHY_RXD1: now reaches U8.24 (RXD1/TXDLY)
- net PHY_RXD1: now also U2.31 (IOT_42b)
- net PHY_RXD0: now reaches U8.25 (RXD0/RXDLY)
- net PHY_RXD0: now also U2.28 (IOT_41a)
- net PHY_RXCTL: now reaches R5.1
- net PHY_RXCTL: now also U2.26 (IOT_39a), U8.26 (RXCTL/PHYAD2); no longer U8.27 (RXC/PHYAD1)
- net PHY_CFG_EXT: now reaches U8.32 (LED0/CFG_EXT)
- net PHY_CFG_EXT: now also D1.2 (A), R8.1
- net PHY_CFG_LDO0: now reaches U8.33 (LED1/CFG_LDO0)
- net PHY_CFG_LDO1: now reaches U8.34 (LED2/CFG_LDO1)
- net PHY_CFG_LDO1: now also D2.2 (A), D3.2 (A), R10.1, R12.2
- net PHY_TXD2: now reaches U2.39 (RGB0)
- new net: D2.1 (K), R11.1
- new net: D1.1 (K), R9.1
- new net: D3.1 (K), R13.2
- new net P3V3: TP21.1
- new net PHY_P3V3: R12.1, R13.1
- no-connect marks 48 -> 27
Other:
- note added: "Configure PHY to use internal LDO at 2.5 V"
- note added: "PHY address is configured as 001"
- note added: "Test Points"
- note added: "Voltage Rails"
- note removed: "PHY address is configured to be 1"
- title: MAX2769B Test Board -> Receiver V0
- moved on the sheet: C40, TP1, TP10, TP11, TP12, TP13, TP14, TP15, TP16, TP17, TP18, TP2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

Commit message: add series resistors to digital signals
Parts:
- added C51, C52: 1u, symbol Device:C_Small
- added C53, C55: 4.7u, symbol Device:C_Small
- added C54, C56: 100n, symbol Device:C_Small
- added R14, R15, R17, R18, R19, R20, R21, R22, R23, R24, R25, R26, R27, R28, R29: 22, symbol Device:R_Small
- added R16: 22, Package_DFN_QFN:QFN-48-1EP_7x7mm_P0.5mm_EP5.6x5.6mm, symbol Device:R_Small
- added TP22: TestPoint, symbol Connector:TestPoint
- added U9: TPS7A20, symbol symbols:TPS7A20
Connections:
- net PHY_P3V3_A is gone; now on net P3V3: U8.11 (AVDD33), U8.40 (AVDD33)
- net PHY_P3V3_D is gone; now on net P3V3: U8.29 (DVDD33)
- net PHY_TXD is gone; now on net PHY_TXD2: U8.16 (TXD2)
- net ADC_I0: now also R16.2; no longer U1.20 (I0)
- net ADC_I1: now also R17.2; no longer U1.21 (I1)
- net ADC_Q0: now also R14.2; no longer U1.18 (Q0)
- net ADC_Q1: now also R15.2; no longer U1.17 (Q1)
- net GND: now also C51.2, C52.2, C53.2, C54.2, C55.2, C56.2, U9. (GND)
- net P3V3: now also C52.1, C53.1, C54.1, C55.1, C56.1, U9.5 (Vout)
- net PHY_RXC: now also R18.1; no longer U8.27 (RXC/PHYAD1)
- net PHY_RXCTL: now also R23.1; no longer U8.26 (RXCTL/PHYAD2)
- net PHY_RXD0: now also R19.1; no longer U8.25 (RXD0/RXDLY)
- net PHY_RXD1: now also R20.1; no longer U8.24 (RXD1/TXDLY)
- net PHY_RXD2: now also R21.1; no longer U8.23 (RXD2/PLLOFF)
- net PHY_RXD3: now also R22.1; no longer U8.22 (RXD3/PHYAD0)
- net PHY_TXC: now also R24.1; no longer U2.35 (IOT_46b_G0)
- net PHY_TXCTL: now also R25.1; no longer U2.36 (IOT_48b)
- net PHY_TXD0: now also R26.1; no longer U2.43 (IOT_49a)
- net PHY_TXD1: now also R28.1; no longer U2.42 (IOT_51a)
- net PHY_TXD2: now also R29.1; no longer U2.39 (RGB0)
- net PHY_TXD3: now also R27.1; no longer U2.38 (IOT_50b)
- net PHY_VDDIO: now also TP22.1
- net VBUS: now also C51.1, U9.1 (Vin), U9.3 (Ven)
- new net: R26.2, U2.43 (IOT_49a)
- new net: R15.1, U1.17 (Q1)
- new net: R27.2, U2.38 (IOT_50b)
- new net: R21.2, U8.23 (RXD2/PLLOFF)
- new net: R22.2, U8.22 (RXD3/PHYAD0)
- new net: R20.2, U8.24 (RXD1/TXDLY)
- new net: R19.2, U8.25 (RXD0/RXDLY)
- new net: R23.2, U8.26 (RXCTL/PHYAD2)
- new net: R18.2, U8.27 (RXC/PHYAD1)
- new net: R28.2, U2.42 (IOT_51a)
- new net: R24.2, U2.35 (IOT_46b_G0)
- new net: R25.2, U2.36 (IOT_48b)
- new net: R14.1, U1.18 (Q0)
- new net: R16.1, U1.20 (I0)
- new net: R17.1, U1.21 (I1)
Other:
- note added: "MCU SPI connector"
- note added: "MCU programming connector - JST/SH"
- note added: "RF IN"
- note added: "Signals"
- moved on the sheet: C2, C22, C23, C27, J1, J3, J4, R2, SW1, TP10, TP11, TP12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

Commit message: mostly finish up PHY schematic
Parts:
- added C57: 100p, symbol Device:C_Small
- added C58, C59: 27p, symbol Device:C_Small
- added J2: RJ45_JK0654219, Connector_RJ:RJ45_Pulse_JK0654219NL_Horizontal, symbol Connector:RJ45_JK0654219
- added R30: 22, symbol Device:R_Small
- added R31: 2.49k, Connector_RJ:RJ45_Pulse_JK0654219NL_Horizontal, symbol Device:R_Small
- added R32, R33: 4.7k, symbol Device:R_Small
- added TP23, TP24, TP25, TP26: TestPoint, symbol Connector:TestPoint
- added Y1: TSX-3225, Package_DFN_QFN:QFN-32-1EP_5x5mm_P0.5mm_EP3.45x3.45mm, symbol Device:Crystal
- R29: footprint (none) -> Connector_RJ:RJ45_Pulse_JK0654219NL_Horizontal
Connections:
- net GND: now also C57.2, C58.2, C59.2, J2.SH, R31.2
- net PHY_CFG_LDO0: now also D3.2 (A), R12.2
- net PHY_CFG_LDO1: no longer D3.2 (A), R12.2
- net PHY_MDC: now also TP23.1, TP25.1
- net PHY_MDIO: now also TP24.1
- net PHY_RXCTL: now also U2.27 (IOT_38b); no longer U2.26 (IOT_39a)
- net PHY_RXD0: now also R32.1
- net PHY_RXD1: now also R33.1
- net PHY_VDDIO: now also R32.2, R33.2
- net at R26.2: now also U2.23 (IOT_37a); no longer U2.43 (IOT_49a)
- net at U2.38 (IOT_50b): no longer R27.2
- net at R29.2: now also U2.43 (IOT_49a)
- net at C5.1: now also R30.2; no longer U1.16 (CLKOUT)
- net PHY_BI_DA_P: now reaches U8.1 (MDIP0)
- net PHY_BI_DA_P: now also J2.11 (MX1+)
- net PHY_BI_DD_N: now reaches U8.10 (MDIN3)
- net PHY_BI_DD_N: now also J2.9 (MX4-)
- net PHY_BI_DA_N: now reaches U8.2 (MDIN0)
- net PHY_BI_DA_N: now also J2.10 (MX1-)
- net PHY_CLK_OUT: now reaches U8.35 (CLK_OUT)
- net PHY_CLK_OUT: now also TP26.1
- net PHY_XTAL_IN: now reaches U8.36 (XTAL_IN)
- net PHY_XTAL_IN: now also C58.1, Y1.1
- net PHY_XTAL_OUT: now reaches U8.37 (XTAL_OUT)
- net PHY_XTAL_OUT: now also C59.1, Y1.2
- net at U8.39 (RSET): now also R31.1
- net PHY_BI_DB_P: now reaches U8.4 (MDIP1)
- net PHY_BI_DB_P: now also J2.4 (MX2+)
- net PHY_BI_DB_N: now reaches U8.5 (MDIN1)
- net PHY_BI_DB_N: now also J2.5 (MX2-)
- net PHY_BI_DC_P: now reaches U8.6 (MDIP2)
- net PHY_BI_DC_P: now also J2.3 (MX3+)
- net PHY_BI_DC_N: now reaches U8.7 (MDIN2)
- net PHY_BI_DC_N: now also J2.2 (MX3-)
- net PHY_BI_DD_P: now reaches U8.9 (MDIP3)
- net PHY_BI_DD_P: now also J2.8 (MX4+)
- net at R28.2: now also U2.25 (IOT_36b); no longer U2.42 (IOT_51a)
- new net: C57.1, J2.1 (MXCT3), J2.12 (MXCT1), J2.6 (MXCT2), J2.7 (MXCT4)
- new net: R27.2, U2.42 (IOT_51a)
- new net: R30.1, U1.16 (CLKOUT)
- no-connect marks 27 -> 37
Other:
- note added: "Configure internal RXC/TXC delay at PHY"
- note added: "Res tolerance should be <1%!"
- moved on the sheet: C1, C10, C11, C12, C13, C14, C15, C16, C17, C18, C19, C20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

Commit message: add pullups
Parts:
- added R34, R35, R36, R37, R38: 4.7k, symbol Device:R_Small
- added R39, R40, R41, R42: 10k, symbol Device:R_Small
- added TP27, TP28, TP29, TP30, TP31: TestPoint, symbol Connector:TestPoint
- added U10, U11: TPS22918, Package_DFN_QFN:Texas_S-PWQFN-N20, symbol symbols:TPS22918
- R31: value 2.49k -> 2.49k 1%; footprint Connector_RJ:RJ45_Pulse_JK0654219NL_Horizontal -> (none)
Connections:
- net CDONE: now also R39.2
- net CRESET_B: now also R40.2
- net GND: now also R34.2, R35.2, R36.2, R37.2, R38.2, U10. (CT), U11. (CT)
- net ICE40_CONFIG_NCS: now also R41.2
- net MAX2769_NIDLE: now also R38.1
- net MAX2769_NSHDN: now also R37.1
- net P1V2: now also U10.1 (VIN); no longer C30.1, C31.1, R3.1, U2.30 (VCC), U2.5 (VCC)
- net PHY_RXD2: now also R34.1
- net SPI_SCK: now also R42.2
- net FPGA_P2V85_EN: now reaches U3.1 (PB9)
- net FPGA_P2V85_EN: now also R35.1, U11. (CT)
- net FPGA_P1V2_EN: now reaches U3.30 (PB6)
- net FPGA_P1V2_EN: now also R36.1, U10. (CT)
- net FPGA_IO2: now reaches U2.4 (IOB_8a)
- net FPGA_IO2: now also TP29.1
- net FPGA_IO1: now reaches U2.45 (IOB_5b)
- net FPGA_IO1: now also TP28.1
- net FPGA_IO0: now reaches U2.48 (IOB_4a)
- net FPGA_IO0: now also TP27.1
- net FPGA_IO3: now reaches U2.26 (IOT_39a)
- net FPGA_IO3: now also TP30.1
- net FPGA_IO4: now reaches U2.38 (IOT_50b)
- net FPGA_IO4: now also TP31.1
- net ICE40_P2V85 renamed P2V85_D
- net P2V85_D: now also U11.1 (VIN); no longer C34.1, C35.1, C36.1, C37.1, C38.1, C39.1, U2.1 (VCCIO_2), U2.22 (SPI_VCCIO1), U2.24 (VPP_2V5), U2.33 (VCCIO_0)
- new net FPGA_P1V2: C30.1, C31.1, R3.1, U10. (CT), U10.6 (Vout), U2.30 (VCC), U2.5 (VCC)
- new net FPGA_P2V85: C34.1, C35.1, C36.1, C37.1, C38.1, C39.1, R39.1, R40.1, R41.1, R42.1, U11. (CT), U11.6 (Vout), U2.1 (VCCIO_2), U2.22 (SPI_VCCIO1), U2.24 (VPP_2V5), U2.33 (VCCIO_0)
- no-connect marks 37 -> 32
Other:
- note added: "Don't turn off PLL automatically"
- note removed: "Res tolerance should be <1%!"
- moved on the sheet: C28, C29, C30, C31, C32, C33, C34, C35, C36, C37, C38, C39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

Commit message: fix SPI bus oversights w/ jumpers
Parts:
- added JP1, JP3, JP5: Jumper_2_Bridged, symbol Jumper:Jumper_2_Bridged
- added JP2, JP4, JP6: Jumper_2_Open, Package_DFN_QFN:WDFN-10-1EP_3x3mm_P0.5mm_EP1.8x2.5mm, symbol Jumper:Jumper_2_Open
- R42: value 10k -> 4.7k
Connections:
- net FPGA_P2V85: no longer R42.1
- net GND: now also R42.2
- net ICE40_CONFIG_NCS: now also JP5.2 (B); no longer R41.2, U2.16 (IOB_35b_SPI_SS)
- net PHY_NRST: now also R42.1
- net SPI_CIPO: now also JP1.2 (B), JP4.2 (B); no longer U2.14 (IOB_32a_SPI_SO)
- net SPI_COPI: now also JP2.2 (B), JP3.2 (B); no longer U2.17 (IOB_33b_SPI_SI)
- net SPI_SCK: no longer R42.2
- new net FLASH_NCS: JP6.2 (B), R41.2
- new net ICE40_SPI_SI: JP3.1 (A), JP4.1 (A), U2.17 (IOB_33b_SPI_SI)
- new net ICE40_SPI_SO: JP1.1 (A), JP2.1 (A), U2.14 (IOB_32a_SPI_SO)
- new net ICE40_SPI_SS: JP5.1 (A), JP6.1 (A), U2.16 (IOB_35b_SPI_SS)
Other:
- moved on the sheet: C30, C31, C32, C33, C34, C35, C36, C37, C38, C39, R3, R35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

Commit message: add flash
Parts:
- added C60: 4.7u, symbol Device:C_Small
- added C61: 100n, symbol Device:C_Small
- added U12: BY25Q16AW, Package_DFN_QFN:Texas_S-PWQFN-N20, symbol symbols:BY25Q16AW
- U3: footprint Package_QFP:LQFP-32_7x7mm_P0.8mm -> LQFP-32_STM
Connections:
- net FLASH_NCS: now also U12.1 (~{CS})
- net FPGA_P1V2: now also U10.5 (QOD); no longer U10. (CT)
- net FPGA_P1V2_EN: now also U10.3 (ON); no longer U10. (CT)
- net FPGA_P2V85: now also U11.5 (QOD); no longer R41.1, U11. (CT)
- net FPGA_P2V85_EN: now also U11.3 (ON); no longer U11. (CT)
- net GND: now also U10.2 (GND), U11.2 (GND), C60.2, C61.2, U12.4 (VSS); no longer U10. (CT), U11. (CT)
- net P2V85_D: now also R41.1, C60.1, C61.1, U12.8 (VCC)
- net SPI_CIPO: now also U12.2 (SO)
- net SPI_COPI: now also U12.5 (SI)
- net SPI_SCK: now also U12.6 (SCLK)
- no-connect marks 32 -> 34
Other:
- note added: "Flash"
- moved on the sheet: C1, C22, C23, C24, C3, C30, C31, C32, C33, C34, C35, C36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

Commit message: start assigning footprints
Parts:
- added C62, C63: 1u, symbol Device:C_Small
- added J5: USB_C_Receptacle_PowerOnly_6P, symbol Connector:USB_C_Receptacle_PowerOnly_6P
- added R43, R44: 5.1k, symbol Device:R_Small
- C27, R10, R11, R8, R9: footprint RF_Module:Digi_XBee_SMT -> (none)
- C40, JP2, JP4, JP6: footprint Package_DFN_QFN:WDFN-10-1EP_3x3mm_P0.5mm_EP1.8x2.5mm -> (none)
- R16: footprint Package_DFN_QFN:QFN-48-1EP_7x7mm_P0.5mm_EP5.6x5.6mm -> (none)
- R29: footprint Connector_RJ:RJ45_Pulse_JK0654219NL_Horizontal -> (none)
- SW1: footprint Package_SON:WSON-8-1EP_6x5mm_P1.27mm_EP3.4x4mm -> (none)
- U1: footprint Package_DFN_QFN:TQFN-28-1EP_5x5mm_P0.5mm_EP2.7x2.7mm -> Package_DFN_QFN:TQFN-28-1EP_5x5mm_P0.5mm_EP3.25x3.25mm
- U10, U11: footprint Package_DFN_QFN:Texas_S-PWQFN-N20 -> Package_TO_SOT_SMD:SOT-23-6
- U12: footprint Package_DFN_QFN:Texas_S-PWQFN-N20 -> Package_SO:SOIC-8_3.9x4.9mm_P1.27mm
- U3: footprint LQFP-32_STM -> Package_QFP:LQFP-32_7x7mm_P0.8mm
- U4, U5, U7, U9: footprint (none) -> Package_TO_SOT_SMD:SOT-23-5
- U6: footprint (none) -> Crystal:Crystal_SMD_WE_CFPX-218-4Pin_2.5x2.0mm
- U8: footprint Package_DFN_QFN:QFN-64-1EP_9x9mm_P0.5mm_EP3.8x3.8mm -> Package_DFN_QFN:QFN-40-1EP_5x5mm_P0.4mm_EP3.6x3.6mm
- Y1: footprint Package_DFN_QFN:QFN-32-1EP_5x5mm_P0.5mm_EP3.45x3.45mm -> Crystal:Crystal_SMD_3225-4Pin_3.2x2.5mm
Connections:
- net GND: now also U4.2 (GND), U5.2 (GND), U7.2 (GND), U9.2 (GND), C62.2, C63.2, J5.A12 (GND), J5.B12 (GND), J5.SH (SHIELD), R43.2, R44.2; no longer U4. (GND), U5. (GND), U7. (GND), U9. (GND)
- net P1V2: now also C62.1
- net P2V85_D: now also C63.1
- net VBUS: now also J5.A9 (VBUS), J5.B9 (VBUS)
- new net: J5.A5 (CC1), R44.1
- new net: J5.B5 (CC2), R43.1
Other:
- moved on the sheet: R35, U11

Commit message: 50 ohm traces
Parts:
- added TP32, TP33: TestPoint, TestPoint:TestPoint_Pad_D1.0mm, symbol Connector:TestPoint
- C1, C10, C11, C12, C13, C14, C15, C16, C17, C18, C19, C2, C20, C21, C22, C23, C24, C25, C26, C27, C28, C29, C3, C30, C31, C32, C33, C34, C35, C36, C37, C38, C39, C4, C40, C41, C42, C43, C44, C45, C46, C47, C48, C49, C5, C50, C51, C52, C53, C54, C55, C56, C57, C58, C59, C6, C60, C61, C62, C63, C7, C8, C9: footprint (none) -> Capacitor_SMD:C_0603_1608Metric
- D1, D2, D3: footprint (none) -> LED_SMD:LED_0805_2012Metric
- J1: footprint (none) -> Connector_Coaxial:SMA_Samtec_SMA-J-P-H-ST-EM1_EdgeMount
- J3: footprint (none) -> Connector_JST:JST_SH_SM03B-SRSS-TB_1x03-1MP_P1.00mm_Horizontal
- J4: footprint (none) -> Connector_PinHeader_2.54mm:PinHeader_1x05_P2.54mm_Vertical
- J5: footprint (none) -> Connector_USB:USB_C_Receptacle_GCT_USB4125-xx-x_6P_TopMnt_Horizontal
- JP1, JP2, JP3, JP4, JP5, JP6: footprint (none) -> Connector_PinHeader_2.54mm:PinHeader_1x02_P2.54mm_Vertical
- R1, R10, R11, R12, R13, R14, R15, R16, R17, R18, R19, R2, R20, R21, R22, R23, R24, R25, R26, R27, R28, R29, R3, R30, R31, R32, R33, R34, R35, R36, R37, R38, R39, R4, R40, R41, R42, R43, R44, R5, R6, R7, R8, R9: footprint (none) -> Resistor_SMD:R_0603_1608Metric
- SW1: footprint (none) -> Button_Switch_THT:SW_PUSH_6mm
- TP1, TP10, TP11, TP12, TP13, TP14, TP15, TP16, TP17, TP18, TP19, TP2, TP20, TP21, TP22, TP23, TP24, TP25, TP26, TP27, TP28, TP29, TP3, TP30, TP31, TP4, TP5, TP6, TP7, TP8, TP9: footprint (none) -> TestPoint:TestPoint_Pad_D1.0mm
Connections:
- net CDONE: now also TP33.1
- net FLASH_NCS: now also TP32.1
