File: max2769test.kicad_sch (KiCad schematic)
At the start: 168 parts, among them J1 Conn_Coaxial, J2 RJ45_JK0654219, J3 Conn_01x03_Socket, J4 Conn_01x05_Pin, J5 USB_C_Receptacle_PowerOnly_6P, SW1 SW_Push, U1 MAX2769B, U10 TPS22918, U11 TPS22918, U12 BY25Q16AW, U2 ICE40UP5K-SG48ITR, U3 STM32C051K6T6, U4 TPS7A20, U5 TPS7A20, U6 TX22-M010S, U7 TPS7A20, U8 RTL8211FD, U9 TPS7A20, Y1 TSX-3225

Commit message: layout start!
Connections:
- net GND: now also U1.29 (EP); no longer U1. (EP)
Changed lines of the file:
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@@
 		(pin "11"
 		)
-		(pin ""
+		(pin "29"
 		)
 		(pin "13"
