File: max2769test.kicad_sch (KiCad schematic)
At the start: 166 parts, among them J1 Conn_Coaxial, J2 RJ45_JK0654219, J3 Conn_01x03_Socket, J4 Conn_01x05_Pin, J5 USB_C_Receptacle_PowerOnly_6P, SW1 SW_Push, U1 MAX2769B, U10 TPS22918, U11 TPS22918, U12 BY25Q16AW, U2 ICE40UP5K-SG48ITR, U3 STM32C051K6T6, U4 TPS7A20, U5 TPS7A20, U6 TX22-M010S, U7 TPS7A20, U8 RTL8211FD, U9 TPS7A20, Y1 TSX-3225

Commit message: sync
Parts:
- removed TP25: TestPoint, TestPoint:TestPoint_Pad_D1.0mm, symbol Connector:TestPoint
- R14, R15, R16, R17: footprint Resistor_SMD:R_0603_1608Metric -> Resistor_SMD:R_0402_1005Metric
Connections:
- net RF_IN: now reaches C2.1, J1.1 (In)
Changed lines of the file:
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@@
 	(wire
 		(pts
-			(xy 88.9 370.84) (xy 92.71 370.84)
-		)
-		(stroke
-			(width 0)
-			(type default)
-		)
-	)
-	(wire
-		(pts
 			(xy 647.7 506.73) (xy 655.32 506.73)
 		)
@@
 		)
 	)
-	(label "PHY_MDC"
-		(at 88.9 370.84 180)
-		(effects
-			(font
-				(size 1.27 1.27)
-			)
-			(justify right bottom)
-		)
-	)
 	(label "ADC_I0"
 		(at 331.47 209.55 0)
@@
 		)
 	)
+	(label "RF_IN"
+		(at 40.64 38.1 0)
+		(effects
+			(font
+				(size 1.27 1.27)
+			)
+			(justify left bottom)
+		)
+	)
 	(label "PHY_RXD3"
 		(at 509.27 438.15 180)
@@
 			)
 		)
-		(property "Footprint" "Resistor_SMD:R_0603_1608Metric"
+		(property "Footprint" "Resistor_SMD:R_0402_1005Metric"
 			(at 297.18 59.69 0)
 			(hide yes)
@@
 			)
 		)
-		(property "Footprint" "Resistor_SMD:R_0603_1608Metric"
+		(property "Footprint" "Resistor_SMD:R_0402_1005Metric"
 			(at 297.18 57.15 0)
 			(hide yes)
@@
 			)
 		)
-		(property "Footprint" "Resistor_SMD:R_0603_1608Metric"
+		(property "Footprint" "Resistor_SMD:R_0402_1005Metric"
 			(at 297.18 62.23 0)
 			(hide yes)
@@
 			)
 		)
-		(property "Footprint" "Resistor_SMD:R_0603_1608Metric"
+		(property "Footprint" "Resistor_SMD:R_0402_1005Metric"
 			(at 297.18 64.77 0)
 			(hide yes)
@@
 					(unit 1)
 				)
-			)
-		)
-	)
-	(symbol
-		(lib_id "Connector:TestPoint")
-		(at 92.71 370.84 270)
-		(unit 1)
-		(body_style 1)
-		(exclude_from_sim no)
-		(in_bom yes)
-		(on_board yes)
-		(in_pos_files yes)
-		(dnp no)
-		(fields_autoplaced yes)
-		(property "Reference" "TP25"
-			(at 97.79 369.5699 90)
-			(show_name no)
-			(do_not_autoplace no)
-			(effects
-				(font
-					(size 1.27 1.27)
-				)
-				(justify left)
-			)
-		)
-		(property "Value" "TestPoint"
-			(at 97.79 372.1099 90)
-			(show_name no)
-			(do_not_autoplace no)
-			(effects
-				(font
-					(size 1.27 1.27)
-				)
-				(justify left)
-			)
-		)
-		(property "Footprint" "TestPoint:TestPoint_Pad_D1.0mm"
-			(at 92.71 375.92 0)
-			(hide yes)
-			(show_name no)
-			(do_not_autoplace no)
-			(effects
-				(font
-					(size 1.27 1.27)
-				)
-			)
-		)
-		(property "Datasheet" ""
-			(at 92.71 375.92 0)
-			(hide yes)
-			(show_name no)
-			(do_not_autoplace no)
-			(effects
-				(font
-					(size 1.27 1.27)
-				)
-			)
-		)
-		(property "Description" "test point"
-			(at 92.71 370.84 0)
-			(hide yes)
-			(show_name no)
-			(do_not_autoplace no)
-			(effects
-				(font
-					(size 1.27 1.27)
-				)
-			)
-		)
-		(pin "1"
-		)
-		(instances
-			(project "max2769test"
-				(path "/e09217dc-f098-45e4-973b-0967150e992c"
-					(reference "TP25")
-					(unit 1)
-				)

Commit message: more layout
Parts:
- removed C5: 10n, Capacitor_SMD:C_0603_1608Metric, symbol Device:C_Small
- removed R28: 22, Resistor_SMD:R_0402_1005Metric, symbol Device:R_Small
- added R45: 22, Resistor_SMD:R_0402_1005Metric, symbol Device:R_Small
- C1, C10, C11, C12, C13, C14, C15, C16, C17, C18, C19, C2, C24, C32, C33, C34, C35, C36, C37, C38, C39: footprint Capacitor_SMD:C_0603_1608Metric -> Capacitor_SMD:C_0402_1005Metric
- R3, R30: footprint Resistor_SMD:R_0603_1608Metric -> Resistor_SMD:R_0402_1005Metric
Connections:
- net ADC_CLK_OUT: now also R30.2
- net FPGA_IO3: now also U2.25 (IOT_36b); no longer U2.26 (IOT_39a)
- net FPGA_IO4: now also U2.23 (IOT_37a); no longer U2.38 (IOT_50b)
- net PHY_RXC: now also U2.26 (IOT_39a); no longer U2.37 (IOT_45a_G1)
- net PHY_TXD1: now also R45.1
- net PHY_TXD2: now also R27.1; no longer R29.1
- net PHY_TXD3: now also R29.1; no longer R27.1
- net at R26.2: now also U2.37 (IOT_45a_G1); no longer U2.23 (IOT_37a)
- new net: R45.2, U2.38 (IOT_50b)
Other:
- moved on the sheet: R26

Commit message: so. much layout oh my g
Parts:
- C30, C31: footprint Capacitor_SMD:C_0603_1608Metric -> Capacitor_SMD:C_0402_1005Metric
- U1: footprint Package_DFN_QFN:TQFN-28-1EP_5x5mm_P0.5mm_EP3.25x3.25mm -> Package_DFN_QFN:TQFN-28-1EP_5x5mm_P0.5mm_EP3.25x3.25mm_ThermalVias
- U8: footprint Package_DFN_QFN:QFN-40-1EP_5x5mm_P0.4mm_EP3.6x3.6mm -> Package_DFN_QFN:QFN-40-1EP_5x5mm_P0.4mm_EP3.6x3.6mm_ThermalVias
Connections:
- net EXT_SPI_CIPO: now also J4.1 (Pin_1); no longer J4.3 (Pin_3)
- net EXT_SPI_COPI: now also J4.3 (Pin_3); no longer J4.2 (Pin_2)
- net EXT_SPI_NCS: now also J4.2 (Pin_2); no longer J4.4 (Pin_4)
- net EXT_SPI_SCK: now also J4.4 (Pin_4); no longer J4.1 (Pin_1)
Changed lines of the file:
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@@
 		)
 	)
-	(label "EXT_SPI_COPI"
+	(label "EXT_SPI_NCS"
 		(at 43.18 68.58 0)
 		(effects
@@
 		)
 	)
-	(label "EXT_SPI_SCK"
+	(label "EXT_SPI_CIPO"
 		(at 43.18 66.04 0)
 		(effects
@@
 		)
 	)
-	(label "EXT_SPI_NCS"
+	(label "EXT_SPI_SCK"
 		(at 43.18 73.66 0)
 		(effects
@@
 		)
 	)
-	(label "EXT_SPI_CIPO"
+	(label "EXT_SPI_COPI"
 		(at 43.18 71.12 0)
 		(effects
@@
 			)
 		)
-		(property "Footprint" "Capacitor_SMD:C_0603_1608Metric"
+		(property "Footprint" "Capacitor_SMD:C_0402_1005Metric"
 			(at 300.99 392.43 0)
 			(hide yes)
@@
 			)
 		)
-		(property "Footprint" "Package_DFN_QFN:QFN-40-1EP_5x5mm_P0.4mm_EP3.6x3.6mm"
+		(property "Footprint" "Package_DFN_QFN:QFN-40-1EP_5x5mm_P0.4mm_EP3.6x3.6mm_ThermalVias"
 			(at 561.34 447.04 0)
 			(hide yes)
@@
 			)
 		)
-		(property "Footprint" "Capacitor_SMD:C_0603_1608Metric"
+		(property "Footprint" "Capacitor_SMD:C_0402_1005Metric"
 			(at 288.29 392.43 0)
 			(hide yes)
@@
 			)
 		)
-		(property "Footprint" "Package_DFN_QFN:TQFN-28-1EP_5x5mm_P0.5mm_EP3.25x3.25mm"
+		(property "Footprint" "Package_DFN_QFN:TQFN-28-1EP_5x5mm_P0.5mm_EP3.25x3.25mm_ThermalVias"
 			(at 256.54 59.69 0)
 			(hide yes)

Commit message: lots of power layout
Parts:
- added C43: 4.7u, Capacitor_SMD:C_0402_1005Metric, symbol Device:C_Small
- added C44: 100n, Capacitor_SMD:C_0402_1005Metric, symbol Device:C_Small
- added TP34, TP35: TestPoint, TestPoint:TestPoint_Pad_D1.0mm, symbol Connector:TestPoint
- U2: footprint Package_DFN_QFN:QFN-48-1EP_7x7mm_P0.5mm_EP5.6x5.6mm -> Package_DFN_QFN:QFN-48-1EP_7x7mm_P0.5mm_EP5.6x5.6mm_ThermalVias
Connections:
- net PHY_P3V3 is gone; now on net P3V3: R12.1, R13.1
- net FPGA_P1V2: now also TP34.1
- net FPGA_P2V85: now also C43.1, C44.1, TP35.1
- net GND: now also C43.2, C44.2
- net PHY_CFG_LDO0: now also D3.1 (K); no longer D3.2 (A)
- net at R13.2: now also D3.2 (A); no longer D3.1 (K)
Other:
- moved on the sheet: C36, C37, D3

Commit message: routed so much..
Parts:
- removed JP1, JP3, JP5: Jumper_2_Bridged, Connector_PinHeader_2.54mm:PinHeader_1x02_P2.54mm_Vertical, symbol Jumper:Jumper_2_Bridged
- removed JP2, JP4: Jumper_2_Open, Connector_PinHeader_2.54mm:PinHeader_1x02_P2.54mm_Vertical, symbol Jumper:Jumper_2_Open
- added J6: Conn_02x02_Odd_Even, Connector_PinHeader_2.54mm:PinHeader_2x02_P2.54mm_Vertical, symbol Connector_Generic:Conn_02x02_Odd_Even
- renumbered JP6 to JP3
Connections:
- net ICE40_CONFIG_NCS is gone; now on net ICE40_SPI_SS: TP6.1, U3.16 (PB1)
- net ICE40_SPI_SI: now also J6.4 (Pin_4)
- net ICE40_SPI_SO: now also J6.1 (Pin_1)
- net PHY_MDC: now also U3.12 (PA5); no longer U3.18 (PA8)
- net SPI_CIPO: now also J6.2 (Pin_2)
- net SPI_COPI: now also J6.3 (Pin_3)
Other:
- moved on the sheet: JP3, R41

Commit message: layout till my eyes bleed
Parts:
- added H1, H2, H3, H4: MountingHole, MountingHole:MountingHole_3.2mm_M3, symbol Mechanical:MountingHole
- C3, C4: footprint Capacitor_SMD:C_0603_1608Metric -> Capacitor_SMD:C_0402_1005Metric
- R1: footprint Resistor_SMD:R_0603_1608Metric -> Resistor_SMD:R_0402_1005Metric

Commit message: so close.. just need to do the cpwg...
Parts:
- removed TP10, TP11, TP12, TP13, TP14, TP15, TP16, TP17, TP18, TP28, TP32, TP33, TP8, TP9: TestPoint, TestPoint:TestPoint_Pad_D1.0mm, symbol Connector:TestPoint
- R32, R33, R34, R5, R6: footprint Resistor_SMD:R_0603_1608Metric -> Resistor_SMD:R_0402_1005Metric
Connections:
- net FPGA_P1V2_EN: now also U3.18 (PA8); no longer U3.30 (PB6)
- net PHY_NRST: now also U3.19 (PA9); no longer U3.27 (PB3)
- net PLL_LOCK_DET: now also U3.7 (PA0); no longer U3.28 (PB4)
