File: max2769test.kicad_pcb (KiCad board)
At the start: 4 copper layers, 166 parts, among them J1 Conn_Coaxial, J2 RJ45_JK0654219, J3 Conn_01x03_Socket, J4 Conn_01x05_Pin, J5 USB_C_Receptacle_PowerOnly_6P, SW1 SW_Push, U1 MAX2769B, U10 TPS22918, U11 TPS22918, U12 BY25Q16AW, U2 ICE40UP5K-SG48ITR, U3 STM32C051K6T6, U4 TPS7A20, U5 TPS7A20, U6 TX22-M010S, U7 TPS7A20, U8 RTL8211FD, U9 TPS7A20, Y1 TSX-3225

Commit message: sync
Parts:
- removed TP25: TestPoint, TestPoint:TestPoint_Pad_D1.0mm
- R14, R15, R16, R17: footprint Resistor_SMD:R_0603_1608Metric -> Resistor_SMD:R_0402_1005Metric
- moved TP22 131.8 mm to (169.2, 91.8)
- moved TP24 119.0 mm to (177.0, 86.6)
- moved TP23 118.6 mm to (179.6, 86.6)
- moved TP20 108.6 mm to (185.8, 94.6)
- moved TP1 66.4 mm to (218.1, 59.8)
- moved TP2 66.4 mm to (218.1, 62.8)
- moved TP27 66.4 mm to (227.2, 75.0)
- moved TP28 66.4 mm to (227.2, 78.0)
- moved TP29 66.4 mm to (230.2, 59.8)
- moved TP3 66.4 mm to (218.1, 65.8)
- moved TP30 66.4 mm to (230.2, 62.8)
- moved TP31 66.4 mm to (230.2, 65.8)
- moved TP32 66.4 mm to (230.2, 68.9)
- moved TP33 66.4 mm to (230.2, 72.0)
- moved TP4 66.4 mm to (218.1, 68.9)
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Connections:
- net Net-(J1-In) renamed /RF_IN
Routing:
- net /PHY_LDO_OUT: track 16.1 -> 54.5 mm, vias 0 -> 5
- net /PHY_MDC: track 0.00 -> 8.63 mm
- net /LNA1_IN: track 0.00 -> 8.55 mm
- net /PHY_MDIO: track 3.98 -> 8.43 mm
- net /PHY_VDDIO: track 25.5 -> 28.7 mm
- net GND: track 21.3 -> 22.4 mm, vias 19 -> 20
- net /RF_IN: track 3.79 -> 4.80 mm

Commit message: more layout
Parts:
- removed C5: 10n, Capacitor_SMD:C_0603_1608Metric
- removed R28: 22, Resistor_SMD:R_0402_1005Metric
- added R45: 22, Resistor_SMD:R_0402_1005Metric, F.Cu at (150.0, 88.8)
- C1, C10, C11, C12, C13, C14, C15, C16, C17, C18, C19, C2, C24, C32, C33, C34, C35, C36, C37, C38, C39: footprint Capacitor_SMD:C_0603_1608Metric -> Capacitor_SMD:C_0402_1005Metric
- R3, R30: footprint Resistor_SMD:R_0603_1608Metric -> Resistor_SMD:R_0402_1005Metric
- moved TP22 134.8 mm to (35.1, 78.5)
- moved R6 128.2 mm to (39.2, 75.3), turned to 0 degrees
- moved C25 110.2 mm to (23.1, 57.8)
- moved C26 110.2 mm to (23.1, 60.3)
- moved C27 110.2 mm to (45.1, 56.5)
- moved U3 110.2 mm to (33.2, 53.0)
- moved TP31 90.1 mm to (149.4, 105.6)
- moved R1 84.3 mm to (129.0, 98.2), turned to -90 degrees
- moved C3 81.5 mm to (130.8, 98.2), turned to -90 degrees
- moved C21 79.1 mm to (136.0, 82.8)
- moved C20 77.4 mm to (136.0, 84.4)
- moved C17 76.2 mm to (142.0, 89.2), turned to -90 degrees
- moved C4 74.4 mm to (127.2, 98.2), turned to 90 degrees
- moved C16 74.3 mm to (140.8, 88.8), turned to -90 degrees
- moved U6 70.7 mm to (139.4, 95.4), turned to 90 degrees
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Connections:
- R26 pad 2: Net-(U2A-IOT_37a) -> Net-(U2A-IOT_45a_G1)
- R27 pad 1: /PHY_TXD3 -> /PHY_TXD2
- R29 pad 1: /PHY_TXD2 -> /PHY_TXD3
- R30 pad 2: Net-(C5-Pad1) -> /ADC_CLK_OUT
- U2 pad 23: Net-(U2A-IOT_37a) -> /FPGA_IO4
- U2 pad 25: Net-(U2A-IOT_36b) -> /FPGA_IO3
- U2 pad 26: /FPGA_IO3 -> /PHY_RXC
- U2 pad 37: /PHY_RXC -> Net-(U2A-IOT_45a_G1)
- U2 pad 38: /FPGA_IO4 -> Net-(U2A-IOT_50b)
Routing:
- net /PHY_TXD3: track 0.00 -> 35.7 mm
- net /PHY_TXD2: track 0.00 -> 33.2 mm
- net /PHY_TXD1: track 0.00 -> 30.7 mm
- net /PHY_TXD0: track 0.00 -> 28.2 mm
- net /PHY_TXCTL: track 0.00 -> 26.1 mm
- net /P2V85_A: track 0.00 -> 25.1 mm, vias 0 -> 2
- net /PHY_TXC: track 0.00 -> 23.6 mm
- net /FPGA_P2V85: track 0.00 -> 18.7 mm
- net /P2V85_D: track 0.00 -> 18.7 mm
- net GND: track 22.4 -> 40.6 mm, vias 20 -> 43
- net /PHY_RXD3: track 4.58 -> 19.6 mm
- net /PHY_RXD2: track 3.98 -> 17.4 mm
- net /PHY_RXD1: track 4.58 -> 17.8 mm
- net /PHY_RXD0: track 5.38 -> 17.4 mm
- net /PHY_RXC: track 5.76 -> 17.1 mm
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- added copper zone on In2.Cu, net (none)
- added copper zone on In1.Cu, net GND

Commit message: so. much layout oh my g
Parts:
- C30, C31: footprint Capacitor_SMD:C_0603_1608Metric -> Capacitor_SMD:C_0402_1005Metric
- U1: footprint Package_DFN_QFN:TQFN-28-1EP_5x5mm_P0.5mm_EP3.25x3.25mm -> Package_DFN_QFN:TQFN-28-1EP_5x5mm_P0.5mm_EP3.25x3.25mm_ThermalVias
- U8: footprint Package_DFN_QFN:QFN-40-1EP_5x5mm_P0.4mm_EP3.6x3.6mm -> Package_DFN_QFN:QFN-40-1EP_5x5mm_P0.4mm_EP3.6x3.6mm_ThermalVias
- moved J4 122.0 mm to (140.2, 128.8), turned to -90 degrees
- moved J3 119.9 mm to (134.9, 147.7), turned to 0 degrees
- moved U3 119.3 mm to (134.6, 115.8)
- moved C26 118.3 mm to (127.6, 115.8), turned to -90 degrees
- moved SW1 118.0 mm to (117.7, 122.6)
- moved C25 117.7 mm to (125.6, 115.8), turned to -90 degrees
- moved C27 102.5 mm to (126.6, 118.8), turned to 180 degrees
- moved J5 101.3 mm to (103.0, 164.2), turned to 0 degrees
- moved TP29 94.9 mm to (142.0, 94.6)
- moved R43 92.0 mm to (104.8, 158.2)
- moved R44 86.4 mm to (101.2, 158.2), turned to 180 degrees
- moved R4 77.3 mm to (89.6, 133.0)
- moved R5 77.3 mm to (87.6, 133.0)
- moved U9 60.8 mm to (76.1, 168.3)
- moved R39 59.7 mm to (78.0, 118.8)
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Connections:
- J4 pad 1: /EXT_SPI_SCK -> /EXT_SPI_CIPO
- J4 pad 2: /EXT_SPI_COPI -> /EXT_SPI_NCS
- J4 pad 3: /EXT_SPI_CIPO -> /EXT_SPI_COPI
- J4 pad 4: /EXT_SPI_NCS -> /EXT_SPI_SCK
Routing:
- net GND: track 40.6 -> 122.5 mm, vias 43 -> 60
- net VBUS: track 0.00 -> 16.1 mm
- net Net-(U3-PF2-NRST): track 0.00 -> 15.4 mm
- net /EXT_SPI_SCK: track 0.00 -> 11.1 mm
- net /EXT_SPI_CIPO: track 0.00 -> 11.0 mm
- net /EXT_SPI_NCS: track 0.00 -> 10.6 mm
- net /P2V85_D: track 18.7 -> 29.0 mm
- net /EXT_SPI_COPI: track 0.00 -> 10.2 mm
- net /FPGA_P1V2: track 3.68 -> 11.7 mm
- net /VCC_TCXO: track 0.00 -> 6.69 mm
- net /P1V2: track 0.00 -> 5.37 mm
- net /PHY_RXD3: track 19.6 -> 16.4 mm
- net Net-(J5-CC2): track 0.00 -> 3.12 mm
- net Net-(J5-CC1): track 0.00 -> 3.12 mm
- net /FPGA_IO2: track 0.00 -> 2.89 mm
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- added copper zone on In2.Cu, net GND
- removed copper zone on In2.Cu, net (none)

Commit message: sync layout
Parts:
- moved SW1 7.55 mm to (125.2, 122.3), turned to -90 degrees
Routing:
- net Net-(U3-PF2-NRST): track 15.4 -> 14.7 mm
Changed lines of the file:
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@@
 	(footprint "Button_Switch_THT:SW_PUSH_6mm"
 		(layer "F.Cu")
-		(at 117.7 122.6)
+		(at 125.25 122.35 -90)
 		(descr "Generic 6mm SW tactile push button")
 		(tags "tact sw push 6mm")
 		(property "Reference" "SW1"
-			(at -2.3 2.4 90)
+			(at 3.25 6.85 90)
 			(layer "F.SilkS")
 			(effects
@@
 		)
 		(property "Value" "SW_Push"
-			(at 3.75 6.7 0)
+			(at 3.75 6.7 90)
 			(layer "F.Fab")
 			(effects
@@
 		)
 		(property "Datasheet" ""
-			(at 0 0 0)
+			(at 0 0 270)
 			(unlocked yes)
 			(layer "F.Fab")
@@
 		)
 		(property "Description" "Push button switch, generic, two pins"
-			(at 0 0 0)
+			(at 0 0 270)
 			(unlocked yes)
 			(layer "F.Fab")
@@
 		(duplicate_pad_numbers_are_jumpers no)
 		(fp_line
-			(start -0.25 1.5)
-			(end -0.25 3)
+			(start 1 5.5)
+			(end 5.5 5.5)
 			(stroke
 				(width 0.12)
@@
 		)
 		(fp_line
-			(start 1 5.5)
-			(end 5.5 5.5)
+			(start 6.75 3)
+			(end 6.75 1.5)
 			(stroke
 				(width 0.12)
@@
 		)
 		(fp_line
-			(start 5.5 -1)
-			(end 1 -1)
+			(start -0.25 1.5)
+			(end -0.25 3)
 			(stroke
 				(width 0.12)
@@
 		)
 		(fp_line
-			(start 6.75 3)
-			(end 6.75 1.5)
+			(start 5.5 -1)
+			(end 1 -1)
 			(stroke
 				(width 0.12)
@@
 		)
 		(fp_line
-			(start -1.5 -1.5)
-			(end -1.25 -1.5)
+			(start -1.5 6)
+			(end -1.25 6)
 			(stroke
 				(width 0.05)
@@
 		)
 		(fp_line
-			(start -1.5 -1.25)
-			(end -1.5 -1.5)
+			(start 7.75 6)
+			(end -1.25 6)
 			(stroke
 				(width 0.05)
@@
 		)
 		(fp_line
-			(start -1.5 5.75)
-			(end -1.5 -1.25)
+			(start 7.75 6)
+			(end 8 6)
 			(stroke
 				(width 0.05)
@@
 		)
 		(fp_line
-			(start -1.5 5.75)
-			(end -1.5 6)
+			(start 8 6)
+			(end 8 5.75)
 			(stroke
 				(width 0.05)
@@
 		)
 		(fp_line
-			(start -1.5 6)
-			(end -1.25 6)
+			(start -1.5 5.75)
+			(end -1.5 6)
 			(stroke
 				(width 0.05)
@@
 		)
 		(fp_line
-			(start -1.25 -1.5)
-			(end 7.75 -1.5)
+			(start -1.5 5.75)
+			(end -1.5 -1.25)
 			(stroke
 				(width 0.05)
@@
 		)
 		(fp_line
-			(start 7.75 -1.5)
-			(end 8 -1.5)
+			(start -1.5 -1.25)
+			(end -1.5 -1.5)
 			(stroke
 				(width 0.05)
@@
 		)
 		(fp_line
-			(start 7.75 6)
-			(end -1.25 6)
+			(start 8 -1.25)
+			(end 8 5.75)
 			(stroke
 				(width 0.05)
@@
 		)
 		(fp_line
-			(start 7.75 6)
-			(end 8 6)
+			(start -1.5 -1.5)
+			(end -1.25 -1.5)
 			(stroke
 				(width 0.05)
@@
 		)
 		(fp_line
-			(start 8 -1.5)
-			(end 8 -1.25)
+			(start -1.25 -1.5)
+			(end 7.75 -1.5)
 			(stroke
 				(width 0.05)
@@
 		)
 		(fp_line
-			(start 8 -1.25)
-			(end 8 5.75)
+			(start 7.75 -1.5)
+			(end 8 -1.5)
 			(stroke
 				(width 0.05)
@@
 		)
 		(fp_line
-			(start 8 6)
-			(end 8 5.75)
+			(start 8 -1.5)
+			(end 8 -1.25)
 			(stroke
 				(width 0.05)
@@
 		)
 		(fp_line
-			(start 0.25 -0.75)
-			(end 3.25 -0.75)
+			(start 0.25 5.25)
+			(end 0.25 -0.75)
 			(stroke
 				(width 0.1)
@@
 		)
 		(fp_line
-			(start 0.25 5.25)
-			(end 0.25 -0.75)
+			(start 6.25 5.25)
+			(end 0.25 5.25)
 			(stroke
 				(width 0.1)
@@
 		)
 		(fp_line
-			(start 3.25 -0.75)
-			(end 6.25 -0.75)
+			(start 0.25 -0.75)
+			(end 3.25 -0.75)
 			(stroke
 				(width 0.1)
@@
 		)
 		(fp_line
-			(start 6.25 -0.75)
-			(end 6.25 5.25)
+			(start 3.25 -0.75)
+			(end 6.25 -0.75)
 			(stroke
 				(width 0.1)
@@
 		)
 		(fp_line
-			(start 6.25 5.25)
-			(end 0.25 5.25)
+			(start 6.25 -0.75)
+			(end 6.25 5.25)
 			(stroke
 				(width 0.1)
@@
 		)
 		(fp_text user "${REFERENCE}"
-			(at 3.25 2.25 0)
+			(at 3.25 2.25 90)
 			(layer "F.Fab")
 			(effects
@@
 		)
 		(pad "1" thru_hole circle
-			(at 0 0 90)
+			(at 0 0)
 			(size 2 2)
 			(drill 1.1)
@@
 		)
 		(pad "1" thru_hole circle
-			(at 6.5 0 90)
+			(at 6.5 0)
 			(size 2 2)
 			(drill 1.1)
@@
 		)
 		(pad "2" thru_hole circle
-			(at 0 4.5 90)
+			(at 0 4.5)
 			(size 2 2)
 			(drill 1.1)
@@
 		)
 		(pad "2" thru_hole circle
-			(at 6.5 4.5 90)
+			(at 6.5 4.5)
 			(size 2 2)
 			(drill 1.1)
@@
 	)
 	(segment
-		(start 124.2 127.1)
-		(end 122.5 127.1)
+		(start 120.75 128.85)
+		(end 120.75 127.15)
 		(width 0.2)
 		(layer "F.Cu")
@@
 	)
 	(segment
-		(start 119.3 127.1)
-		(end 119.4 127.2)
+		(start 120.75 123.95)
+		(end 120.65 124.05)
 		(width 0.2)
 		(layer "F.Cu")
@@
 	)
 	(segment
-		(start 117.7 127.1)
-		(end 119.3 127.1)
+		(start 120.75 122.35)
+		(end 120.75 123.95)
 		(width 0.2)
 		(layer "F.Cu")
@@
 	)
 	(segment
-		(start 122.5 127.1)
-		(end 122.4 127.2)
+		(start 120.75 127.15)
+		(end 120.65 127.05)
 		(width 0.2)
 		(layer "F.Cu")
@@
 	)
 	(via
-		(at 119.4 127.2)
+		(at 120.65 124.05)
 		(size 0.6)
 		(drill 0.3)
@@
 	)
 	(via
-		(at 122.4 127.2)
+		(at 120.65 127.05)
 		(size 0.6)
 		(drill 0.3)
@@
 	)
 	(segment
-		(start 117.7 122.6)
-		(end 124.2 122.6)
+		(start 125.25 122.35)
+		(end 127.375 120.225)
 		(width 0.2)
 		(layer "F.Cu")
@@
 	)
 	(segment
-		(start 127.375 119.425)
-		(end 127.375 118.8)
+		(start 125.25 122.35)
+		(end 125.25 128.85)
 		(width 0.2)
 		(layer "F.Cu")
@@
 	)
 	(segment
-		(start 127.375 118.8)
-		(end 129.175 117)
+		(start 127.375 120.225)
+		(end 127.375 118.8)
 		(width 0.2)
 		(layer "F.Cu")
@@
 	)
 	(segment
-		(start 129.175 117)
-		(end 130.425 117)
+		(start 127.375 118.8)
+		(end 129.175 117)
 		(width 0.2)
 		(layer "F.Cu")
@@
 	)
 	(segment
-		(start 124.2 122.6)
-		(end 127.375 119.425)
+		(start 129.175 117)
+		(end 130.425 117)
 		(width 0.2)
 		(layer "F.Cu")

Commit message: small sync just to bring up to date
Parts:
- moved C63 66.1 mm to (113.6, 105.0)
- moved U11 66.1 mm to (117.4, 105.0)
- moved R35 66.1 mm to (114.6, 108.0)
Changed lines of the file:
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@@
 	(footprint "Resistor_SMD:R_0603_1608Metric"
 		(layer "F.Cu")
-		(at 141.975 168.2 180)
+		(at 114.6 108 180)
 		(descr "Resistor SMD 0603 (1608 Metric), square (rectangular) end terminal, IPC-7351 nominal, (Body size source: IPC-SM-782 page 72, https://www.pcb-3d.com/wordpress/wp-content/uploads/ipc-sm-782a_amendment_1_and_2.pdf)")
 		(tags "resistor")
@@
 	(footprint "Package_TO_SOT_SMD:SOT-23-6"
 		(layer "F.Cu")
-		(at 144.7375 165.15)
+		(at 117.3625 104.95)
 		(descr "SOT, 6 Pin (JEDEC MO-178 Var AB https://www.jedec.org/document_search?search_api_views_fulltext=MO-178)")
 		(tags "SOT TO_SOT_SMD")
@@
 	(footprint "Capacitor_SMD:C_0603_1608Metric"
 		(layer "F.Cu")
-		(at 140.975 165.175 -90)
+		(at 113.6 104.975 -90)
 		(descr "Capacitor SMD 0603 (1608 Metric), square (rectangular) end terminal, IPC-7351 nominal, (Body size source: IPC-SM-782 page 76, https://www.pcb-3d.com/wordpress/wp-content/uploads/ipc-sm-782a_amendment_1_and_2.pdf)")
 		(tags "capacitor")
@@
 	)
 	(segment
-		(start 140.975 166)
-		(end 141.15 166.175)
+		(start 113.6 105.8)
+		(end 113.775 105.975)
 		(width 0.2)
 		(layer "F.Cu")
@@
 	)
 	(segment
-		(start 140.975 165.95)
-		(end 141.775 165.15)
+		(start 113.6 105.75)
+		(end 114.4 104.95)
 		(width 0.2)
 		(layer "F.Cu")
@@
 	)
 	(segment
-		(start 140.975 165.95)
-		(end 140.975 166)
+		(start 113.6 105.75)
+		(end 113.6 105.8)
 		(width 0.2)
 		(layer "F.Cu")
@@
 	)
 	(segment
-		(start 141.15 166.175)
-		(end 141.15 168.2)
+		(start 113.775 105.975)
+		(end 113.775 108)
 		(width 0.2)
 		(layer "F.Cu")
@@
 	)
 	(segment
-		(start 141.775 165.15)
-		(end 143.6 165.15)
+		(start 114.4 104.95)
+		(end 116.225 104.95)
 		(width 0.2)
 		(layer "F.Cu")
@@
 	)
 	(segment
-		(start 142.8 168.2)
-		(end 142.8 166.9)
+		(start 115.425 108)
+		(end 115.425 106.7)
 		(width 0.2)
 		(layer "F.Cu")
@@
 	)
 	(segment
-		(start 142.8 166.9)
-		(end 143.6 166.1)
+		(start 115.425 106.7)
+		(end 116.225 105.9)
 		(width 0.2)
 		(layer "F.Cu")
@@
 	)
 	(segment
-		(start 140.975 164.4)
-		(end 143.4 164.4)
+		(start 113.6 104.2)
+		(end 116.025 104.2)
 		(width 0.2)
 		(layer "F.Cu")
@@
 	)
 	(segment
-		(start 143.4 164.4)
-		(end 143.6 164.2)
+		(start 116.025 104.2)
+		(end 116.225 104)
 		(width 0.2)
 		(layer "F.Cu")

Commit message: lots of power layout
Parts:
- added C43: 4.7u, Capacitor_SMD:C_0402_1005Metric, F.Cu at (143.2, 91.8)
- added C44: 100n, Capacitor_SMD:C_0402_1005Metric, F.Cu at (144.2, 91.0)
- added TP34: TestPoint, TestPoint:TestPoint_Pad_D1.0mm, F.Cu at (162.0, 103.6)
- added TP35: TestPoint, TestPoint:TestPoint_Pad_D1.0mm, F.Cu at (151.2, 81.8)
- U2: footprint Package_DFN_QFN:QFN-48-1EP_7x7mm_P0.5mm_EP5.6x5.6mm -> Package_DFN_QFN:QFN-48-1EP_7x7mm_P0.5mm_EP5.6x5.6mm_ThermalVias
- moved C51 109.6 mm to (163.0, 106.7)
- moved C52 109.6 mm to (170.6, 106.7)
- moved U9 109.6 mm to (166.9, 106.8)
- moved C6 79.3 mm to (123.0, 86.6)
- moved C7 79.3 mm to (115.4, 86.6)
- moved U4 79.3 mm to (119.2, 86.6)
- moved R37 73.1 mm to (120.8, 71.0)
- moved R38 73.1 mm to (120.8, 73.5)
- moved R36 67.5 mm to (159.8, 106.6), turned to -90 degrees
- moved U10 64.5 mm to (156.6, 104.0), turned to 90 degrees
- moved JP1 63.2 mm to (154.6, 126.0)
- moved JP6 63.2 mm to (177.6, 126.0)
- moved JP2 63.2 mm to (159.2, 126.0)
- moved JP3 63.2 mm to (163.8, 126.0)
- moved JP4 63.2 mm to (168.4, 126.0)
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Connections:
- D3 pad 1: Net-(D3-K) -> /PHY_CFG_LDO0
- D3 pad 2: /PHY_CFG_LDO0 -> Net-(D3-A)
- R12 pad 1: /PHY_P3V3 -> /P3V3
- R13 pad 1: /PHY_P3V3 -> /P3V3
- R13 pad 2: Net-(D3-K) -> Net-(D3-A)
Routing:
- net /P3V3: track 20.3 -> 136.9 mm, vias 0 -> 4
- net /PHY_CFG_LDO0: track 1.97 -> 61.8 mm, vias 1 -> 2
- net /PHY_CFG_LDO1: track 3.34 -> 60.8 mm, vias 1 -> 2
- net /FPGA_P2V85: track 16.7 -> 74.1 mm, vias 0 -> 5
- net /PHY_CFG_EXT: track 2.74 -> 55.9 mm, vias 1 -> 2
- net /P2V85_A: track 27.8 -> 59.3 mm, vias 2 -> 6
- net /FPGA_P1V2: track 11.7 -> 42.5 mm, vias 0 -> 3
- net /SWCLK: track 0.00 -> 18.8 mm
- net /SWDIO: track 0.00 -> 16.0 mm
- net GND: track 122.5 -> 131.0 mm, vias 60 -> 70
- net /LNA1_IN: track 9.30 -> 3.30 mm
- net /PHY_VDDIO: track 20.2 -> 23.9 mm
- net /PHY_LDO_OUT: track 55.1 -> 51.5 mm
- net Net-(D3-A): track 0.00 -> 2.64 mm
- net Net-(D2-K): track 0.00 -> 2.44 mm
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Other:
- board outline added: 125.8 x 55.4 mm
- board text added: "1000M"
- board text added: "100M"
- board text added: "10M"

Commit message: routed so much..
Parts:
- removed JP1, JP5: Jumper_2_Bridged, Connector_PinHeader_2.54mm:PinHeader_1x02_P2.54mm_Vertical
- removed JP2, JP4: Jumper_2_Open, Connector_PinHeader_2.54mm:PinHeader_1x02_P2.54mm_Vertical
- removed the JP3 at (163.8, 126.0)
- added J6: Conn_02x02_Odd_Even, Connector_PinHeader_2.54mm:PinHeader_2x02_P2.54mm_Vertical, F.Cu at (168.2, 112.5)
- moved C28 88.5 mm to (143.7, 110.1)
- moved C29 88.5 mm to (151.7, 110.1)
- moved U7 88.5 mm to (147.9, 110.2)
- moved J5 68.2 mm to (110.6, 96.4), turned to -90 degrees
- moved R44 65.4 mm to (116.6, 94.6), turned to 90 degrees
- moved R43 61.1 mm to (116.6, 98.2), turned to -90 degrees
- moved U12 49.2 mm to (160.6, 113.2), turned to 180 degrees
- moved C61 43.7 mm to (160.4, 117.0)
- moved C60 38.6 mm to (160.4, 118.8)
- moved JP3 9.87 mm to (170.7, 118.9), turned to -90 degrees
- moved TP24 4.65 mm to (179.4, 84.0)
- moved TP26 3.01 mm to (179.0, 107.8)
- moved C30 1.79 mm to (142.0, 98.8)
- moved C31 1.79 mm to (140.8, 98.8)
- renumbered JP6 to JP3
Connections:
- TP6 pad 1: /ICE40_CONFIG_NCS -> /ICE40_SPI_SS
- U3 pad 12: unconnected-(U3-PA5-Pad12) -> /PHY_MDC
- U3 pad 16: /ICE40_CONFIG_NCS -> /ICE40_SPI_SS
- U3 pad 18: /PHY_MDC -> unconnected-(U3-PA8-Pad18)
Routing:
- net /PHY_MDC: track 8.95 -> 94.7 mm, vias 0 -> 2
- net /PHY_MDIO: track 10.4 -> 94.0 mm, vias 0 -> 2
- net /ICE40_SPI_SS: track 0.00 -> 80.4 mm, vias 0 -> 1
- net /SPI_COPI: track 0.00 -> 69.4 mm, vias 0 -> 2
- net /SPI_SCK: track 0.00 -> 68.3 mm, vias 0 -> 4
- net VBUS: track 16.1 -> 73.9 mm
- net /MAX2769_NCS: track 0.00 -> 40.4 mm, vias 0 -> 2
- net /ICE40_SPI_SI: track 0.00 -> 34.1 mm, vias 0 -> 1
- net /ICE40_SPI_SO: track 0.00 -> 31.8 mm, vias 0 -> 1
- net /CRESET_B: track 0.00 -> 26.0 mm, vias 0 -> 2
- net /CDONE: track 0.00 -> 20.0 mm, vias 0 -> 2
- net GND: track 131.0 -> 149.2 mm, vias 70 -> 76
- net /SPI_CIPO: track 0.00 -> 15.3 mm
- net /FLASH_NCS: track 0.00 -> 6.68 mm
- net /P1V2: track 5.37 -> 10.8 mm
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- added copper zone on F.Cu, net GND

Commit message: mounting holes
Parts:
- added H1: MountingHole, MountingHole:MountingHole_3.2mm_M3, F.Cu at (229.4, 79.2)
- added H2: MountingHole, MountingHole:MountingHole_3.2mm_M3, F.Cu at (110.8, 79.2)
- added H3: MountingHole, MountingHole:MountingHole_3.2mm_M3, F.Cu at (110.8, 127.4)
- added H4: MountingHole, MountingHole:MountingHole_3.2mm_M3, F.Cu at (229.4, 127.4)
- moved C18 0.89 mm to (135.0, 96.0)
- moved C19 0.89 mm to (136.2, 96.0)
- moved R16 0.40 mm to (139.0, 87.2)
- moved R17 0.40 mm to (139.0, 86.0)
Routing:
- net /MAX2769_NIDLE: track 2.24 -> 62.8 mm, vias 1 -> 2
- net /MAX2769_NSHDN: track 0.00 -> 46.6 mm, vias 0 -> 2
- net /FPGA_P2V85: track 74.1 -> 71.8 mm
- net /P2V85_D: track 33.4 -> 35.0 mm
Other:
- board text added: "AZ"
