File: max2769test.kicad_pcb (KiCad board)
At the start: 4 copper layers, 125.8 x 55.4 mm, 168 parts, among them J1 Conn_Coaxial, J2 RJ45_JK0654219, J3 Conn_01x03_Socket, J4 Conn_01x05_Pin, J5 USB_C_Receptacle_PowerOnly_6P, J6 Conn_02x02_Odd_Even, SW1 SW_Push, U1 MAX2769B, U10 TPS22918, U11 TPS22918, U12 BY25Q16AW, U2 ICE40UP5K-SG48ITR, U3 STM32C051K6T6, U4 TPS7A20, U5 TPS7A20, U6 TX22-M010S, U7 TPS7A20, U8 RTL8211FD, U9 TPS7A20, Y1 TSX-3225

Commit message: layout till my eyes bleed
Parts:
- C3, C4: footprint Capacitor_SMD:C_0603_1608Metric -> Capacitor_SMD:C_0402_1005Metric
- R1: footprint Resistor_SMD:R_0603_1608Metric -> Resistor_SMD:R_0402_1005Metric
- moved R6 125.7 mm to (163.8, 92.2), turned to 180 degrees
- moved R41 88.4 mm to (164.0, 118.0), turned to 90 degrees
- moved R5 84.1 mm to (163.8, 97.4), turned to 180 degrees
- moved R4 83.8 mm to (167.2, 101.4)
- moved R40 50.8 mm to (142.2, 105.0)
- moved R38 48.5 mm to (142.2, 117.0), turned to -90 degrees
- moved R39 46.2 mm to (139.2, 100.4), turned to -90 degrees
- moved R37 21.9 mm to (122.8, 92.8), turned to 180 degrees
- moved J1 13.4 mm to (132.4, 64.6)
- moved H1 13.2 mm to (229.4, 66.0)
- moved H2 13.2 mm to (110.8, 66.0)
- moved C20 2.84 mm to (138.8, 84.6)
- moved C21 2.84 mm to (138.8, 83.0)
- moved R16 1.40 mm to (140.4, 87.2)
- moved R17 1.40 mm to (140.4, 86.0)
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Routing:
- net /FPGA_P2V85_EN: track 2.43 -> 39.1 mm, vias 0 -> 2
- net /FPGA_P2V85: track 71.8 -> 90.7 mm, vias 5 -> 6
- net /RF_IN: track 4.86 -> 17.9 mm
- net /PHY_VDDIO: track 25.9 -> 36.3 mm, vias 2 -> 3
- net /P2V85_D: track 35.0 -> 41.3 mm
- net GND: track 149.2 -> 143.8 mm, vias 76 -> 74
- net /MAX2769_NIDLE: track 62.8 -> 65.7 mm
- net /FLASH_NCS: track 6.68 -> 9.13 mm
- net /PHY_RXD3: track 16.4 -> 18.9 mm
- net /MAX2769_NSHDN: track 46.6 -> 48.8 mm
- net /CDONE: track 20.0 -> 22.1 mm
- net /PHY_RXCTL: track 16.4 -> 18.3 mm
- net /PHY_RXC: track 16.2 -> 18.0 mm
- net /CRESET_B: track 26.0 -> 27.8 mm
- net /P2V85_A: track 59.3 -> 60.8 mm
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- removed copper zone on F.Cu, net GND
Other:
- board size 125.8 x 55.4 mm -> 125.8 x 68.6 mm
- board text removed: "AZ"

Commit message: so close.. just need to do the cpwg...
Parts:
- removed TP10, TP11, TP12, TP13, TP14, TP15, TP16, TP17, TP18, TP28, TP32, TP33, TP8, TP9: TestPoint, TestPoint:TestPoint_Pad_D1.0mm
- C10, C11, TP27: moved to B.Cu
- R32, R33, R34, R5, R6: footprint Resistor_SMD:R_0603_1608Metric -> Resistor_SMD:R_0402_1005Metric
- moved TP22 140.2 mm to (175.2, 82.0)
- moved TP3 139.2 mm to (111.4, 88.0)
- moved TP1 127.9 mm to (123.0, 82.0)
- moved TP4 124.2 mm to (131.6, 107.8)
- moved TP30 115.3 mm to (153.2, 101.2)
- moved TP19 113.5 mm to (147.2, 105.6)
- moved TP27 113.5 mm to (145.2, 88.8), turned to 180 degrees
- moved TP2 106.4 mm to (143.6, 78.6)
- moved TP5 104.0 mm to (155.0, 114.0)
- moved R34 96.0 mm to (163.4, 91.4), turned to 180 degrees
- moved R33 93.4 mm to (163.6, 93.6), turned to 180 degrees
- moved R32 91.5 mm to (163.6, 95.8), turned to 180 degrees
- moved TP6 88.6 mm to (173.8, 119.0)
- moved TP21 88.4 mm to (173.0, 108.8), turned to -90 degrees
- moved TP7 83.7 mm to (173.8, 112.4), turned to -90 degrees
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Connections:
- U3 pad 18: unconnected-(U3-PA8-Pad18) -> /FPGA_P1V2_EN
- U3 pad 19: unconnected-(U3-PA9-Pad19) -> /PHY_NRST
- U3 pad 27: /PHY_NRST -> unconnected-(U3-PB3-Pad27)
- U3 pad 28: /PLL_LOCK_DET -> unconnected-(U3-PB4-Pad28)
- U3 pad 30: /FPGA_P1V2_EN -> unconnected-(U3-PB6-Pad30)
- U3 pad 7: unconnected-(U3-PA0-Pad7) -> /PLL_LOCK_DET
Routing:
- net VBUS: track 73.9 -> 173.0 mm, vias 0 -> 2
- net /P2V85_D: track 41.3 -> 139.7 mm, vias 0 -> 7
- net /PHY_NRST: track 4.64 -> 101.3 mm, vias 0 -> 2
- net /FPGA_P1V2_EN: track 2.59 -> 69.0 mm, vias 0 -> 2
- net /PLL_LOCK_DET: track 0.00 -> 46.8 mm, vias 0 -> 2
- net /PHY_VDDIO: track 36.3 -> 46.1 mm, vias 3 -> 5
- net GND: track 143.8 -> 149.4 mm
- net /P1V2: track 10.8 -> 15.5 mm
- net /FPGA_IO0: track 0.00 -> 4.09 mm, vias 0 -> 1
- net /P3V3: track 135.1 -> 138.9 mm
- net /PHY_RXD2: track 16.2 -> 19.5 mm
- net /P2V85_A: track 60.8 -> 64.0 mm, vias 6 -> 5
- net /ICE40_SPI_SS: track 80.4 -> 83.5 mm
- net /SPI_CIPO: track 15.3 -> 18.3 mm
- net /FPGA_IO3: track 0.00 -> 2.88 mm
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
Commit message: finally no more drc errors
Parts:
- added G***: LOGO, LOGO, F.Cu at (214.4, 74.0)
- moved C2 1.06 mm to (132.4, 84.2)
Routing:
- net /RF_IN: track 17.9 -> 19.4 mm
- net /LNA1_IN: track 3.30 -> 1.97 mm
- net GND: vias 74 -> 92
- added copper zone on B.Cu, net GND
- added copper zone on F.Cu, net GND
Other:
- board text added: "PNTSDR V0 2026 Oct Adrian Zhang"
