File: _restore_backup_2026-10-04T21-34-31-541/max2769test.kicad_sch (KiCad schematic)
At the start: 166 parts, among them J1 Conn_Coaxial, J2 RJ45_JK0654219, J3 Conn_01x03_Socket, J4 Conn_01x05_Pin, J5 USB_C_Receptacle_PowerOnly_6P, SW1 SW_Push, U1 MAX2769B, U10 TPS22918, U11 TPS22918, U12 BY25Q16AW, U2 ICE40UP5K-SG48ITR, U3 STM32C051K6T6, U4 TPS7A20, U5 TPS7A20, U6 TX22-M010S, U7 TPS7A20, U8 RTL8211FD, U9 TPS7A20, Y1 TSX-3225

Commit message: work on PHY layout
Parts:
- removed C64: 100p, Capacitor_SMD:C_0603_1608Metric, symbol Device:C_Small
- removed C65: 4.7u, Capacitor_SMD:C_0402_1005Metric, symbol Device:C_Small
- removed C66: 100n, Capacitor_SMD:C_0402_1005Metric, symbol Device:C_Small
Connections:
- net PHY_BI_DB_N: now also J2.5 (MX2-); no longer J2.4 (MX2+)
- net PHY_BI_DB_P: now also J2.4 (MX2+); no longer J2.5 (MX2-)
- net PHY_BI_DD_N: now also J2.9 (MX4-); no longer J2.8 (MX4+)
- net PHY_BI_DD_P: now also J2.8 (MX4+); no longer J2.9 (MX4-)
- net at C57.1, J2.1 (MXCT3), J2.7 (MXCT4): now also J2.12 (MXCT1), J2.6 (MXCT2)
Other:
- note added: "PHY pin 29"
- note added: "PHY pin 40"
